File: 7-SEG_DISP.kicad_sch (KiCad schematic)
At the start: 18 parts, among them J12 Conn_01x08, J13 Conn_01x04, U2 74F573SC, U3 74F573SC, U4 74F573SC, U5 SC39-12EWA, U6 SC39-12EWA, U7 SC39-12EWA, U8 74F573SC, U9 SC39-12EWA

Commit message: power
Parts:
- J12: footprint (none) -> Connector_PinHeader_2.54mm:PinHeader_1x08_P2.54mm_Vertical
- J13: footprint (none) -> Connector_PinHeader_2.54mm:PinHeader_1x04_P2.54mm_Vertical
- U2, U3, U4, U8: footprint SOIC20_12P7X5P4_ONS -> (none)
- U5, U6, U7, U9: footprint Display_7Segment:Sx39-1xxxxx -> (none)
Connections:
- net +5V: now also U2.20 (VCC), U3.20 (VCC), U4.20 (VCC), U8.20 (VCC)
