File: INT.kicad_sch (KiCad schematic)
At the start: 4 parts, among them SW2 SW_Push_Dual, SW3 SW_Push_Dual

Commit message: power
Parts:
- C6, C7: footprint (none) -> Capacitor_SMD:C_1206_3216Metric_Pad1.33x1.80mm_HandSolder
Changed lines of the file:
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@@
 	)
 	(label "P3.2"
-		(at 109.22 90.17 0)
+		(at 109.22 72.39 0)
 		(effects
 			(font
@@
 	)
 	(label "P3.3"
-		(at 134.62 78.74 0)
+		(at 134.62 72.39 0)
 		(effects
 			(font
@@
 			)
 		)
-		(property "Footprint" ""
+		(property "Footprint" "Capacitor_SMD:C_1206_3216Metric_Pad1.33x1.80mm_HandSolder"
 			(at 129.54 108.9152 0)
 			(effects
@@
 			)
 		)
-		(property "Footprint" ""
+		(property "Footprint" "Capacitor_SMD:C_1206_3216Metric_Pad1.33x1.80mm_HandSolder"
 			(at 96.52 108.9152 0)
 			(effects
