File: LCD.kicad_sch (KiCad schematic)
At the start: 4 parts, among them J10 LCM-S01602DTR_M, J11 Conn_01x03, J9 Conn_01x08

Commit message: power
Parts:
- J10: footprint LCM-S01602DTR_M:LCD_LCM-S01602DTR_M -> imports:LCD_LCM-S01602DTR_M
- J11: footprint (none) -> Connector_PinHeader_2.54mm:PinHeader_1x03_P2.54mm_Vertical
- J9: footprint (none) -> Connector_PinHeader_2.54mm:PinHeader_1x08_P2.54mm_Vertical
- RV1: footprint (none) -> imports:601030_AVX
Changed lines of the file:
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@@
 			)
 		)
-		(property "Footprint" ""
+		(property "Footprint" "Connector_PinHeader_2.54mm:PinHeader_1x03_P2.54mm_Vertical"
 			(at 175.26 72.39 0)
 			(effects
@@
 			)
 		)
-		(property "Footprint" ""
+		(property "Footprint" "Connector_PinHeader_2.54mm:PinHeader_1x08_P2.54mm_Vertical"
 			(at 120.65 71.12 0)
 			(effects
@@
 			)
 		)
-		(property "Footprint" "LCM-S01602DTR_M:LCD_LCM-S01602DTR_M"
+		(property "Footprint" "imports:LCD_LCM-S01602DTR_M"
 			(at 151.13 71.12 0)
 			(effects
@@
 			)
 		)
-		(property "Footprint" ""
+		(property "Footprint" "imports:601030_AVX"
 			(at 185.42 57.15 0)
 			(effects
