File: PWR.kicad_sch (KiCad schematic)
At the start: 0 parts

Commit message: power
Parts:
- added C10, C11: 0.1uF, Capacitor_SMD:C_1206_3216Metric_Pad1.33x1.80mm_HandSolder, symbol Device:C
- added C8: 10uF, Capacitor_SMD:C_1206_3216Metric_Pad1.33x1.80mm_HandSolder, symbol Device:C
- added C9: 1uF, Capacitor_SMD:C_1206_3216Metric_Pad1.33x1.80mm_HandSolder, symbol Device:C
- added D2: LED, symbol Device:LED
- added J14: PJ-102A, Connector_BarrelJack:BarrelJack_CUI_PJ-102AH_Horizontal, symbol PJ-102A:PJ-102A
- added J15, J16: Conn_01x01, Connector_PinHeader_2.54mm:PinHeader_1x01_P2.54mm_Vertical, symbol Connector_Generic:Conn_01x01
- added Q1: LM7805CT_NOPB, imports:TO254P1054X470X2600-3, symbol LM7805CT_NOPB:LM7805CT_NOPB
- added R2, R3: 2, Resistor_SMD:R_1206_3216Metric_Pad1.30x1.75mm_HandSolder, symbol Device:R
- added R4: 150, Resistor_SMD:R_1206_3216Metric_Pad1.30x1.75mm_HandSolder, symbol Device:R
- added SW20: SW_Nidec_CAS-120A1, symbol Switch:SW_Nidec_CAS-120A1
- added U10: 2SA2222SG, imports:TO-220F-3SG_15P87X10P16_ONS, symbol 2025-09-25_04-52-18:2SA2222SG
Connections:
- new net: C10.1, C8.1, C9.1, R2.1, R3.1, SW20.3 (A), U10.3 (E)
- new net: Q1.1 (IN), R2.2, R3.2, U10.1 (B)
- new net: J14.1, SW20.2 (B)
- new net: D2.2 (A), R4.2
- new net +5V: C11.1, J16.1 (Pin_1), Q1.3 (OUT), R4.1, U10.2 (C)
- new net GND: C10.2, C11.2, C8.2, C9.2, D2.1 (K), J14.2, J14.3, J15.1 (Pin_1), Q1.2 (GND)
- no-connect marks 0 -> 1
