File: 8051 Breakout Board/8051_breakout.kicad_sch (KiCad schematic)
At the start: 18 parts, among them J1 Conn_01x20, J2 Conn_01x20, J3 Conn_02x03_Counter_Clockwise, SW1 SW_Push_Dual, U1 AT89S51-24PU, Y1 ABL-11.0592MHZ-B1U-T

Commit message: traces
Parts:
- H1, H2, H3, H4: footprint MountingHole:MountingHole_2.2mm_M2_DIN965 -> MountingHole:MountingHole_2.2mm_M2_DIN965_Pad
Changed lines of the file:
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@@
 			)
 		)
-		(property "Footprint" "MountingHole:MountingHole_2.2mm_M2_DIN965"
+		(property "Footprint" "MountingHole:MountingHole_2.2mm_M2_DIN965_Pad"
 			(at 234.95 50.8 0)
 			(effects
@@
 			)
 		)
-		(property "Footprint" "MountingHole:MountingHole_2.2mm_M2_DIN965"
+		(property "Footprint" "MountingHole:MountingHole_2.2mm_M2_DIN965_Pad"
 			(at 234.95 63.5 0)
 			(effects
@@
 			)
 		)
-		(property "Footprint" "MountingHole:MountingHole_2.2mm_M2_DIN965"
+		(property "Footprint" "MountingHole:MountingHole_2.2mm_M2_DIN965_Pad"
 			(at 234.95 57.15 0)
 			(effects
@@
 			)
 		)
-		(property "Footprint" "MountingHole:MountingHole_2.2mm_M2_DIN965"
+		(property "Footprint" "MountingHole:MountingHole_2.2mm_M2_DIN965_Pad"
 			(at 234.95 44.45 0)
 			(effects
