File: 8051 Breakout Board/8051_breakout.kicad_pcb (KiCad board)
At the start: 2 copper layers, 55.9 x 83.8 mm, 18 parts, among them J1 Conn_01x20, J2 Conn_01x20, J3 Conn_02x03_Counter_Clockwise, SW1 SW_Push_Dual, U1 AT89S51-24PU, Y1 ABL-11.0592MHZ-B1U-T

Commit message: traces
Parts:
- added kibuzzard-68D5B3C4: G***, kibuzzard-68D5B3C4, F.Cu at (111.8, 132.7)
- H1, H2, H3, H4: footprint MountingHole:MountingHole_2.2mm_M2_DIN965 -> MountingHole:MountingHole_2.2mm_M2_DIN965_Pad
- moved SW1 2.23 mm to (93.3, 56.2)
- moved C1 1.27 mm to (132.1, 58.4)
- moved C4 1.27 mm to (121.9, 58.4)
- moved D2 1.27 mm to (127.0, 58.4)
- moved R1 1.27 mm to (124.5, 58.4)
- moved R4 1.27 mm to (129.5, 58.4)
Routing:
- net +5V: track 65.3 -> 104.5 mm
- net /RST: track 85.2 -> 91.7 mm, vias 0 -> 1
- net /XTAL1: track 23.0 -> 22.5 mm
- net GND: vias 6 -> 262
Other:
- board text added: "AD0 AD1 AD2 AD3 AD4 AD5 AD6 AD7 A15 A14 A13 A12 A11 A10 A9 A8"
- board text added: "GND MOSI VCC"
- board text added: "MOSI MISO SCK RXD TXD INT0 INT1 T0 T1 WR RD"
- board text added: "P1.0 P1.1 P1.2 P1.3 P1.4 P1.5 P1.6 P1.7 RST P3.0 P3.1 P3.2 P3.3 P3.4 P3.5 P3.6 P3.7 XTAL2 XTAL1 GND"
- board text added: "RST SCK MISO"
- board text added: "VCC P0.0 P0.1 P0.2 P0.3 P0.4 P0.5 P0.6 P0.7 EA ALE PSEN P2.7 P2.6 P2.5 P2.4 P2.3 P2.2 P2.1 P2.0"
- board text removed: "AT89S51 Breakout Board"

Commit message: silkscreen bs
Parts:
- added G***: LOGO, LOGO, F.Cu at (92.7, 128.3)
- added kibuzzard-68D5FACE: G***, kibuzzard-68D5FACE, F.Cu at (130.8, 127.0)

Commit message: done
Parts:
- added ?: , clipboard:b3f230c9-10c0-4d2b-a50d-c1d3223b5fd3, B.Cu at (91.4, 58.4)
- added ?: , clipboard:b4713e84-af34-4575-aedb-29b788b1340b, B.Cu at (112.9, 62.6)
- added ?: , clipboard:a52bedb4-97ff-4e76-972c-cf4dcddbd37b, B.Cu at (104.1, 123.7)
- added ?: , clipboard:67966e1b-97d9-4a56-a0fe-5229392e6668, B.Cu at (121.3, 67.6)
- added ?: , clipboard:aac07f4e-c2d1-4b1e-b003-b98e1c51be95, B.Cu at (107.2, 56.2)
- added ?: , clipboard:3740d66f-e0a3-4d38-9639-7d3d28e194a3, B.Cu at (138.6, 61.5)
- added ?: , clipboard:62ec4081-8ac1-45e2-9960-4b9c9dfd804b, B.Cu at (135.5, 126.1)
- added ?: , clipboard:b4713e84-af34-4575-aedb-29b788b1340b, B.Cu at (153.0, 61.3)
- added ?: , clipboard:d386838b-1032-4213-a0d3-9db035365056, B.Cu at (120.1, 139.6)
- added ?: , clipboard:63c00108-0446-4b83-a5cd-419c989de34f, B.Cu at (80.2, 130.6)
- added ?: , clipboard:5b28d9ec-89ab-48fd-9efa-5624283c358b, B.Cu at (124.0, 53.3)
- added ?: , clipboard:62ec4081-8ac1-45e2-9960-4b9c9dfd804b, B.Cu at (107.6, 77.1)
- added ?: , clipboard:13cca798-ea0b-493d-bdc4-b2d1531b002e, B.Cu at (123.3, 129.6)
- added ?: , clipboard:13b4419b-8654-49d9-8ec1-5027561bad04, B.Cu at (103.0, 77.2)
- added ?: , clipboard:dc2016ff-9d75-4c92-a41a-f960c426ace3, B.Cu at (101.7, 44.1)
- added G***: LOGO, LOGO, B.Cu at (111.3, 105.2)
