File: 8051 Development Board/7-SEG_DISP.kicad_sch (KiCad schematic)
At the start: 18 parts, among them J12 Conn_01x08, J13 Conn_01x04, U2 74F573SC, U3 74F573SC, U4 74F573SC, U5 SC39-12EWA, U6 SC39-12EWA, U7 SC39-12EWA, U8 74F573SC, U9 SC39-12EWA

Commit message: layout
Parts:
- U2, U3, U4: footprint (none) -> imports:SOIC20_12P7X5P4_ONS
- U5: renamed from U8; footprint (none) -> imports:SOIC20_12P7X5P4_ONS
- U6: renamed from U5; footprint (none) -> Display_7Segment:7SegmentLED_LTS6760_LTS6780
- U7: renamed from U6; footprint (none) -> Display_7Segment:7SegmentLED_LTS6760_LTS6780
- U8: renamed from U7; footprint (none) -> Display_7Segment:7SegmentLED_LTS6760_LTS6780
- U9: footprint (none) -> Display_7Segment:7SegmentLED_LTS6760_LTS6780
Changed lines of the file:
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@@
 		(dnp no)
 		(fields_autoplaced yes)
-		(property "Reference" "U7"
+		(property "Reference" "U8"
 			(at 180.34 33.0199 90)
 			(effects
@@
 			)
 		)
-		(property "Footprint" ""
+		(property "Footprint" "Display_7Segment:7SegmentLED_LTS6760_LTS6780"
 			(at 180.34 34.29 0)
 			(effects
@@
 			(project "8051"
 				(path "/1fd5cb60-9043-4003-959b-0153e5ed66c7/dd62a08f-b237-46a3-8243-a8f19a82c583"
-					(reference "U7")
+					(reference "U8")
 					(unit 1)
 				)
@@
 		(on_board yes)
 		(dnp no)
-		(fields_autoplaced yes)
 		(property "Reference" "U2"
 			(at 81.28 88.8999 90)
@@
 			)
 		)
-		(property "Footprint" ""
+		(property "Footprint" "imports:SOIC20_12P7X5P4_ONS"
 			(at 52.07 110.49 0)
 			(effects
@@
 			)
 		)
-		(property "Footprint" ""
+		(property "Footprint" "Display_7Segment:7SegmentLED_LTS6760_LTS6780"
 			(at 233.68 34.29 0)
 			(effects
@@
 		(dnp no)
 		(fields_autoplaced yes)
-		(property "Reference" "U5"
+		(property "Reference" "U6"
 			(at 73.66 33.0199 90)
 			(effects
@@
 			)
 		)
-		(property "Footprint" ""
+		(property "Footprint" "Display_7Segment:7SegmentLED_LTS6760_LTS6780"
 			(at 73.66 34.29 0)
 			(effects
@@
 			(project ""
 				(path "/1fd5cb60-9043-4003-959b-0153e5ed66c7/dd62a08f-b237-46a3-8243-a8f19a82c583"
-					(reference "U5")
+					(reference "U6")
 					(unit 1)
 				)
@@
 		(dnp no)
 		(fields_autoplaced yes)
-		(property "Reference" "U8"
+		(property "Reference" "U5"
 			(at 241.3 88.8999 90)
 			(effects
@@
 			)
 		)
-		(property "Footprint" ""
+		(property "Footprint" "imports:SOIC20_12P7X5P4_ONS"
 			(at 212.09 110.49 0)
 			(effects
@@
 			(project "8051"
 				(path "/1fd5cb60-9043-4003-959b-0153e5ed66c7/dd62a08f-b237-46a3-8243-a8f19a82c583"
-					(reference "U8")
+					(reference "U5")
 					(unit 1)
 				)
@@
 			)
 		)
-		(property "Footprint" ""
+		(property "Footprint" "imports:SOIC20_12P7X5P4_ONS"
 			(at 105.41 110.49 0)
 			(effects
@@
 		(dnp no)
 		(fields_autoplaced yes)
-		(property "Reference" "U6"
+		(property "Reference" "U7"
 			(at 127 33.0199 90)
 			(effects
@@
 			)
 		)
-		(property "Footprint" ""
+		(property "Footprint" "Display_7Segment:7SegmentLED_LTS6760_LTS6780"
 			(at 127 34.29 0)
 			(effects
@@
 			(project "8051"
 				(path "/1fd5cb60-9043-4003-959b-0153e5ed66c7/dd62a08f-b237-46a3-8243-a8f19a82c583"
-					(reference "U6")
+					(reference "U7")
 					(unit 1)
 				)
@@
 			)
 		)
-		(property "Footprint" ""
+		(property "Footprint" "imports:SOIC20_12P7X5P4_ONS"
 			(at 158.75 110.49 0)
 			(effects
