File: 8051 Development Board/INT.kicad_sch (KiCad schematic)
At the start: 4 parts, among them SW2 SW_Push_Dual, SW3 SW_Push_Dual

Commit message: layout
Parts:
- SW2, SW3: footprint (none) -> Button_Switch_THT:SW_PUSH_6mm_H7.3mm
Changed lines of the file:
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@@
 		(at 120.65 90.17)
 	)
-	(bus_entry
-		(at 106.68 68.58)
-		(size 2.54 2.54)
-		(stroke
-			(width 0)
-			(type default)
-		)
-	)
-	(bus_entry
-		(at 132.08 68.58)
-		(size 2.54 2.54)
-		(stroke
-			(width 0)
-			(type default)
-		)
-	)
 	(wire
 		(pts
@@
 		)
 	)
-	(bus
-		(pts
-			(xy 99.06 68.58) (xy 106.68 68.58)
-		)
-		(stroke
-			(width 0)
-			(type default)
-		)
-	)
 	(wire
 		(pts
@@
 		)
 	)
-	(bus
-		(pts
-			(xy 106.68 68.58) (xy 132.08 68.58)
-		)
-		(stroke
-			(width 0)
-			(type default)
-		)
-	)
 	(wire
 		(pts
@@
 		)
 	)
-	(bus
-		(pts
-			(xy 132.08 68.58) (xy 138.43 68.58)
-		)
-		(stroke
-			(width 0)
-			(type default)
-		)
-	)
 	(wire
 		(pts
@@
 		)
 	)
-	(label "P3.2"
-		(at 109.22 72.39 0)
+	(hierarchical_label "P3.3"
+		(shape input)
+		(at 134.62 72.39 90)
 		(effects
 			(font
 				(size 1.27 1.27)
 			)
-			(justify left bottom)
-		)
-	)
-	(label "P3.[0..7]"
-		(at 138.43 68.58 0)
+			(justify left)
+		)
+	)
+	(hierarchical_label "P3.2"
+		(shape input)
+		(at 109.22 72.39 90)
 		(effects
 			(font
 				(size 1.27 1.27)
 			)
-			(justify left bottom)
-		)
-	)
-	(label "P3.3"
-		(at 134.62 72.39 0)
-		(effects
-			(font
-				(size 1.27 1.27)
-			)
-			(justify left bottom)
-		)
-	)
-	(hierarchical_label "P3"
-		(shape input)
-		(at 99.06 68.58 180)
-		(effects
-			(font
-				(size 1.27 1.27)
-			)
-			(justify right)
+			(justify left)
 		)
 	)
@@
 			)
 		)
-		(property "Footprint" ""
+		(property "Footprint" "Button_Switch_THT:SW_PUSH_6mm_H7.3mm"
 			(at 125.73 100.33 0)
 			(effects
@@
 			)
 		)
-		(property "Footprint" ""
+		(property "Footprint" "Button_Switch_THT:SW_PUSH_6mm_H7.3mm"
 			(at 100.33 100.33 0)
 			(effects
