File: 8051 Development Board/LCD.kicad_sch (KiCad schematic)
At the start: 4 parts, among them J10 LCM-S01602DTR_M, J11 Conn_01x03, J9 Conn_01x08

Commit message: layout
Connections:
- no-connect marks 0 -> 2
Changed lines of the file:
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@@
 		(color 0 0 0 0)
+	)
+	(no_connect
+		(at 163.83 88.9)
+	)
+	(no_connect
+		(at 163.83 86.36)
 	)
 	(wire
