File: 8051 Development Board/ISP.kicad_sch (KiCad schematic)
At the start: 0 parts

Commit message: layout
Parts:
- added C4: 10u, Capacitor_SMD:C_0805_2012Metric_Pad1.18x1.45mm_HandSolder, symbol Device:C
- added J6: Conn_02x03_Counter_Clockwise, Connector_PinHeader_2.54mm:PinHeader_2x03_P2.54mm_Vertical, symbol Connector_Generic:Conn_02x03_Counter_Clockwise
- added R1: 10k, Resistor_SMD:R_0805_2012Metric_Pad1.20x1.40mm_HandSolder, symbol Device:R
- added SW1: SW_Push_Dual, Button_Switch_THT:SW_PUSH_6mm_H7.3mm, symbol Switch:SW_Push
Connections:
- new net (MISO)P1.6: J6.3 (Pin_3)
- new net (MOSI)P1.5: J6.5 (Pin_5)
- new net (SCK)P1.7: J6.2 (Pin_2)
- new net +5V: J6.4 (Pin_4), SW1.1
- new net GND: C4.2, J6.6 (Pin_6), R1.1
- new net RST: C4.1, J6.1 (Pin_1), R1.2, SW1.2

Commit message: 5v power plane
Parts:
- C4: footprint Capacitor_SMD:C_0805_2012Metric_Pad1.18x1.45mm_HandSolder -> Capacitor_SMD:C_1206_3216Metric_Pad1.33x1.80mm_HandSolder
- R1: footprint Resistor_SMD:R_0805_2012Metric_Pad1.20x1.40mm_HandSolder -> Resistor_SMD:R_1206_3216Metric_Pad1.30x1.75mm_HandSolder
Changed lines of the file:
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@@
 			)
 		)
-		(property "Footprint" "Capacitor_SMD:C_0805_2012Metric_Pad1.18x1.45mm_HandSolder"
+		(property "Footprint" "Capacitor_SMD:C_1206_3216Metric_Pad1.33x1.80mm_HandSolder"
 			(at 162.2552 90.17 0)
 			(effects
@@
 			)
 		)
-		(property "Footprint" "Resistor_SMD:R_0805_2012Metric_Pad1.20x1.40mm_HandSolder"
+		(property "Footprint" "Resistor_SMD:R_1206_3216Metric_Pad1.30x1.75mm_HandSolder"
 			(at 150.368 86.36 90)
 			(effects
