File: 8051 Development Board/8051.kicad_sch (KiCad schematic)
At the start: 11 parts, among them J1 Conn_01x08, J2 Conn_02x03_Counter_Clockwise, J3 Conn_01x08, J4 Conn_01x08, J5 Conn_01x08, U1 AT89S51-24PU, Y1 ABL-11.0592MHZ-B1U-T

Commit message: layout
Parts:
- added H1, H2, H3, H4: MountingHole, MountingHole:MountingHole_2.2mm_M2_DIN965_Pad, symbol Mechanical:MountingHole
- Y1: footprint (none) -> Crystal:Crystal_HC49-4H_Vertical
Other:
- sheet INT ports: added P3.2, P3.3; removed P3
- sheet ISP ports: added (MISO)P1.6, (MOSI)P1.5, (SCK)P1.7; removed MISO, MOSI, SCK

Commit message: layout
Parts:
- removed J2: Conn_02x03_Counter_Clockwise, Connector_PinHeader_2.54mm:PinHeader_2x03_P2.54mm_Vertical, symbol Connector_Generic:Conn_02x03_Counter_Clockwise
Connections:
- net MISO is gone; now on net P1.6: U1.7 ((MISO)_P1.6)
- net MOSI is gone; now on net P1.5: U1.6 ((MOSI)_P1.5)
- net SCK is gone; now on net P1.7: U1.8 ((SCK)_P1.7)
Changed lines of the file:
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@@
-	(wire
-		(pts
-			(xy 83.82 67.31) (xy 83.82 73.66)
-		)
-		(stroke
-			(width 0)
-			(type default)
-		)
-	)
 	(wire
 		(pts
@@
 	(wire
 		(pts
-			(xy 86.36 86.36) (xy 86.36 92.71)
-		)
-		(stroke
-			(width 0)
-			(type default)
-		)
-	)
-	(wire
-		(pts
 			(xy 172.72 90.17) (xy 194.31 90.17)
 		)
@@
 	(wire
 		(pts
-			(xy 83.82 86.36) (xy 83.82 95.25)
+			(xy 83.82 67.31) (xy 83.82 95.25)
 		)
 		(stroke
@@
 	(wire
 		(pts
-			(xy 86.36 67.31) (xy 86.36 73.66)
+			(xy 86.36 67.31) (xy 86.36 92.71)
 		)
 		(stroke
@@
 	(wire
 		(pts
-			(xy 88.9 67.31) (xy 88.9 73.66)
+			(xy 88.9 67.31) (xy 88.9 90.17)
 		)
 		(stroke
@@
 		(pts
 			(xy 214.63 92.71) (xy 220.98 92.71)
-		)
-		(stroke
-			(width 0)
-			(type default)
-		)
-	)
-	(wire
-		(pts
-			(xy 88.9 86.36) (xy 88.9 90.17)
 		)
 		(stroke
@@
 		)
 	)
+	(label "P1.7"
+		(at 46.99 95.25 0)
+		(effects
+			(font
+				(size 1.27 1.27)
+			)
+			(justify left bottom)
+		)
+	)
 	(label "P0.[0..7]"
 		(at 212.09 78.74 180)
@@
 		)
 	)
-	(label "MOSI"
-		(at 50.8 90.17 180)
-		(effects
-			(font
-				(size 1.27 1.27)
-			)
-			(justify right bottom)
-		)
-	)
 	(label "P2.7"
 		(at 177.8 107.95 180)
@@
 		)
 	)
-	(label "SCK"
-		(at 50.8 95.25 180)
-		(effects
-			(font
-				(size 1.27 1.27)
-			)
-			(justify right bottom)
-		)
-	)
 	(label "P3.7"
 		(at 101.6 118.11 0)
@@
 		)
 	)
-	(label "MISO"
-		(at 50.8 92.71 180)
-		(effects
-			(font
-				(size 1.27 1.27)
-			)
-			(justify right bottom)
-		)
-	)
 	(label "P2.2"
 		(at 177.8 120.65 180)
@@
 		)
 	)
+	(label "P1.5"
+		(at 46.99 90.17 0)
+		(effects
+			(font
+				(size 1.27 1.27)
+			)
+			(justify left bottom)
+		)
+	)
 	(label "P1.[0..7]"
 		(at 102.87 64.77 0)
@@
 			)
 			(justify right bottom)
+		)
+	)
+	(label "P1.6"
+		(at 46.99 92.71 0)
+		(effects
+			(font
+				(size 1.27 1.27)
+			)
+			(justify left bottom)
 		)
 	)
@@
 					(unit 1)
 				)
-			)
-		)
-	)
-	(symbol
-		(lib_id "Connector_Generic:Conn_02x03_Counter_Clockwise")
-		(at 86.36 78.74 90)
-		(mirror x)
-		(unit 1)
-		(exclude_from_sim no)
-		(in_bom yes)
-		(on_board yes)
-		(dnp no)
-		(property "Reference" "J2"
-			(at 81.28 78.7399 90)
-			(effects
-				(font
-					(size 1.27 1.27)
-				)
-				(justify left)
-			)
-		)
-		(property "Value" "Conn_02x03_Counter_Clockwise"
-			(at 81.28 81.2799 90)
-			(effects
-				(font
-					(size 1.27 1.27)
-				)
-				(justify left)
-			)
-		)
-		(property "Footprint" "Connector_PinHeader_2.54mm:PinHeader_2x03_P2.54mm_Vertical"
-			(at 86.36 78.74 0)
-			(effects
-				(font
-					(size 1.27 1.27)
-				)
-				(hide yes)
-			)
-		)
-		(property "Datasheet" "~"
-			(at 86.36 78.74 0)
-			(effects
-				(font
-					(size 1.27 1.27)
-				)
-				(hide yes)
-			)
-		)
-		(property "Description" "Generic connector, double row, 02x03, counter clockwise pin numbering scheme (similar to DIP package numbering), script generated (kicad-library-utils/schlib/autogen/connector/)"
-			(at 86.36 78.74 0)
-			(effects
-				(font
-					(size 1.27 1.27)
-				)
-				(hide yes)
-			)
-		)
-		(pin "6"
-		)
-		(pin "4"
-		)
-		(pin "3"
-		)
-		(pin "2"
-		)
-		(pin "5"
-		)
-		(pin "1"
-		)
-		(instances
-			(project ""
-				(path "/1fd5cb60-9043-4003-959b-0153e5ed66c7"
-					(reference "J2")
-					(unit 1)
-				)

Commit message: dev board gerbers
Parts:
- removed H1, H2, H3, H4: MountingHole, MountingHole:MountingHole_2.2mm_M2_DIN965_Pad, symbol Mechanical:MountingHole
