File: 8051 Development Board/PWR.kicad_sch (KiCad schematic)
At the start: 14 parts, among them J14 PJ-102A, J15 Conn_01x01, J16 Conn_01x01, Q1 LM7805CT_NOPB, SW20 SW_Nidec_CAS-120A1, U10 2SA2222SG

Commit message: layout
Parts:
- D2: footprint (none) -> LED_THT:LED_D3.0mm
- SW20: footprint (none) -> imports:500SSP1S1M2QEA
Connections:
- net VIN: now reaches J14.1, SW20.2 (B)
Changed lines of the file:
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@@
+		)
+	)
+	(label "VIN"
+		(at 57.15 85.09 0)
+		(effects
+			(font
+				(size 1.27 1.27)
+			)
+			(justify left bottom)
 		)
 	)
@@
 			)
 		)
-		(property "Footprint" ""
+		(property "Footprint" "imports:500SSP1S1M2QEA"
 			(at 69.85 95.25 0)
 			(effects
@@
 			)
 		)
-		(property "Footprint" ""
+		(property "Footprint" "LED_THT:LED_D3.0mm"
 			(at 186.69 110.49 0)
 			(effects

Commit message: resistors
Parts:
- R2, R3: value 2 -> 20
Changed lines of the file:
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@@
 			)
 		)
-		(property "Value" "2"
+		(property "Value" "20"
 			(at 115.57 68.5799 0)
 			(effects
@@
 			)
 		)
-		(property "Value" "2"
+		(property "Value" "20"
 			(at 100.33 68.5799 0)
 			(effects
