File: 8051 Development Board v2/8051.kicad_pcb (KiCad board)
At the start: 2 copper layers, 128.3 x 125.7 mm, 75 parts, among them J1 Conn_01x08, J10 LCM-S01602DTR_M, J11 Conn_01x03, J12 Conn_01x08, J13 Conn_01x04, J14 PJ-102A, J15 Conn_01x01, J16 Conn_01x01, J3 Conn_01x08, J4 Conn_01x08, J5 Conn_01x08, J6 Conn_02x03_Counter_Clockwise, J8 Conn_01x08, J9 Conn_01x08, Q1 LM7805CT_NOPB, SW1 SW_Push_Dual, SW10 SW_Push_Dual, SW11 SW_Push_Dual, SW12 SW_Push_Dual, SW13 SW_Push_Dual, SW14 SW_Push_Dual, SW15 SW_Push_Dual, SW16 SW_Push_Dual, SW17 SW_Push_Dual, SW18 SW_Push_Dual, SW19 SW_Push_Dual, SW2 SW_Push_Dual, SW20 SW_Nidec_CAS-120A1, SW3 SW_Push_Dual, SW4 SW_Push_Dual, SW5 SW_Push_Dual, SW6 SW_Push_Dual, SW7 SW_Push_Dual, SW8 SW_Push_Dual, SW9 SW_Push_Dual, U1 AT89S51-24PU, U10 2SA2222SG, U2 74F573SC, U3 74F573SC, U4 74F573SC, U5 74F573SC, U6 SC39-12EWA, U7 SC39-12EWA, U8 SC39-12EWA, U9 SC39-12EWA, Y1 ABL-11.0592MHZ-B1U-T

Commit message: ultra
Parts:
- removed C1, C10, C11: 0.1uF, Capacitor_SMD:C_1206_3216Metric_Pad1.33x1.80mm_HandSolder
- removed C2, C3: 30pF, Capacitor_SMD:C_1206_3216Metric_Pad1.33x1.80mm_HandSolder
- removed C4: 10u, Capacitor_SMD:C_1206_3216Metric_Pad1.33x1.80mm_HandSolder
- removed C6, C7, C9: 1uF, Capacitor_SMD:C_1206_3216Metric_Pad1.33x1.80mm_HandSolder
- removed C8: 10uF, Capacitor_SMD:C_1206_3216Metric_Pad1.33x1.80mm_HandSolder
- removed D2: LED, LED_THT:LED_D3.0mm
- removed G*** (x2): LOGO, LOGO
- removed J1, J12, J3, J4, J5, J8, J9: Conn_01x08, Connector_PinHeader_2.54mm:PinHeader_1x08_P2.54mm_Vertical
- removed J10: LCM-S01602DTR_M, imports:LCD_LCM-S01602DTR_M
- removed J11: Conn_01x03, Connector_PinHeader_2.54mm:PinHeader_1x03_P2.54mm_Vertical
- removed J13: Conn_01x04, Connector_PinHeader_2.54mm:PinHeader_1x04_P2.54mm_Vertical
- removed J14: PJ-102A, Connector_BarrelJack:BarrelJack_CUI_PJ-102AH_Horizontal
- removed J15, J16: Conn_01x01, Connector_PinHeader_2.54mm:PinHeader_1x01_P2.54mm_Vertical
- removed J6: Conn_02x03_Counter_Clockwise, Connector_PinHeader_2.54mm:PinHeader_2x03_P2.54mm_Vertical
- removed Q1: LM7805CT_NOPB, imports:TO254P1054X470X2600-3
- removed R1: 10k, Resistor_SMD:R_1206_3216Metric_Pad1.30x1.75mm_HandSolder
- removed R2, R3: 2, Resistor_SMD:R_1206_3216Metric_Pad1.30x1.75mm_HandSolder
- removed R4: 150, Resistor_SMD:R_1206_3216Metric_Pad1.30x1.75mm_HandSolder
- removed RN1: R_Network08_US, Resistor_THT:R_Array_SIP9
- removed RN2, RN3, RN4, RN5, RN6, RN7, RN8, RN9: R_Pack04_SIP, Resistor_THT:R_Array_SIP8
- removed RV1: 601030, imports:601030_AVX
- removed SW1, SW10, SW11, SW12, SW13, SW14, SW15, SW16, SW17, SW18, SW19, SW2, SW3, SW4, SW5, SW6, SW7, SW8, SW9: SW_Push_Dual, Button_Switch_THT:SW_PUSH_6mm_H7.3mm
- removed SW20: SW_Nidec_CAS-120A1, imports:500SSP1S1M2QEA
- removed U1: AT89S51-24PU, imports:40P6_ATM
- removed U10: 2SA2222SG, imports:TO-220F-3SG_15P87X10P16_ONS
- removed U2, U3, U4, U5: 74F573SC, imports:SOIC20_12P7X5P4_ONS
- removed U6, U7, U8, U9: SC39-12EWA, Display_7Segment:7SegmentLED_LTS6760_LTS6780
- removed Y1: ABL-11.0592MHZ-B1U-T, Crystal:Crystal_HC49-4H_Vertical
- removed kibuzzard-68D8BB38: G***, kibuzzard-68D8BB38
- removed kibuzzard-68D8BC51: G***, kibuzzard-68D8BC51
Routing:
- net /KEYPAD_HEX/C4: track 109.9 -> 0.00 mm
- net +5V: track 109.7 -> 0.00 mm, vias 4 -> 0
- net /KEYPAD_HEX/C3: track 95.3 -> 0.00 mm
- net /KEYPAD_HEX/R1: track 88.4 -> 0.00 mm
- net Net-(J12-Pin_4): track 87.0 -> 0.00 mm, vias 3 -> 0
- net Net-(J12-Pin_3): track 86.4 -> 0.00 mm, vias 4 -> 0
- net Net-(J12-Pin_8): track 84.4 -> 0.00 mm, vias 5 -> 0
- net Net-(J12-Pin_6): track 84.1 -> 0.00 mm, vias 4 -> 0
- net /P3.3: track 83.5 -> 0.00 mm
- net Net-(J12-Pin_1): track 83.2 -> 0.00 mm, vias 3 -> 0
- net Net-(J12-Pin_7): track 82.5 -> 0.00 mm, vias 4 -> 0
- net /LCD/D7: track 81.4 -> 0.00 mm
- net Net-(J12-Pin_2): track 80.8 -> 0.00 mm, vias 4 -> 0
- net Net-(J12-Pin_5): track 80.7 -> 0.00 mm, vias 4 -> 0
- net /KEYPAD_HEX/C2: track 80.5 -> 0.00 mm
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- removed copper zone on F.Cu, net +5V
- removed copper zone on B.Cu, net GND
Other:
- board outline removed
- board text removed: "2SA2222SG"
- board text removed: "601030"
- board text removed: "7-20V"
- board text removed: "74F573SC"
- board text removed: "7_SEG_DISP"
- board text removed: "ABL-11.0592MHZ-B1U-T"
- board text removed: "AT89S51"
- board text removed: "C1 C2 C3 C4 R1 R2 R3 R4"
- board text removed: "D7 D6 D5 D4 D3 D2 D1 D0"
- board text removed: "E RW RS"
- board text removed: "GND 5V"
- board text removed: "GND MOSI VCC"
- board text removed: "KEYPAD_HEX"
- board text removed: "LCD"
- board text removed: "LCM-S01602DTR/M"
- board text removed: "LM7805CT"
- board text removed: "P0.0 P0.1 P0.2 P0.3 P0.4 P0.5 P0.6 P0.7 P2.7 P2.6 P2.5 P2.4 P2.3 P2.2 P2.1 P2.0"
- board text removed: "P1.0 P1.1 P1.2 P1.3 P1.4 P1.5 P1.6 P1.7 P3.0 P3.1 P3.2 P3.3 P3.4 P3.5 P3.6 P3.7"
- board text removed: "Port 0"
- board text removed: "Port 1"
- board text removed: "Port 2"
- board text removed: "Port 3"
- board text removed: "RESET"
- board text removed: "RST SCK MISO"
