File: 8051 Development Board v2/ADC.kicad_sch (KiCad schematic)
At the start: 2 parts, among them J7 Conn_02x06_Counter_Clockwise, U11 MCP3008

Commit message: nets
Parts:
- removed J7: Conn_02x06_Counter_Clockwise, symbol Connector_Generic:Conn_02x06_Counter_Clockwise
- added C5: 100n, Capacitor_SMD:C_1206_3216Metric, symbol Device:C
- added J15: Conn_02x05_Counter_Clockwise, symbol Connector_Generic:Conn_02x05_Counter_Clockwise
- added R99: R, Resistor_SMD:R_1206_3216Metric, symbol Device:R
- added RP1: R_Photo, symbol Device:R_Photo
- added RV2: 10k, symbol Device:R_Potentiometer
- added U12: LM35-LP, Package_TO_SOT_THT:TO-92_Inline, symbol Sensor_Temperature:LM35-LP
Connections:
- net +5V: now also C5.1, RP1.1, RV2.1, U12.1 (+V_{S})
- net GND: now also C5.2, R99.2, RV2.3, U12.3 (GND)
- net CH0: now reaches U11.1 (CH0)
- net CH0: now also J15.10 (Pin_10)
- net at U11.10 (~{CS}/SHDN): now also J15.4 (Pin_4)
- net at U11.11 (Din): now also J15.3 (Pin_3)
- net at U11.12 (Dout): now also J15.2 (Pin_2)
- net at U11.13 (CLK): now also J15.1 (Pin_1)
- net CH1: now reaches U11.2 (CH1)
- net CH1: now also J15.9 (Pin_9)
- net CH2: now reaches U11.3 (CH2)
- net CH2: now also J15.8 (Pin_8)
- net CH3: now reaches U11.4 (CH3)
- net CH3: now also J15.7 (Pin_7)
- net CH4: now reaches U11.5 (CH4)
- net CH4: now also J15.6 (Pin_6)
- net CH5: now reaches U11.6 (CH5)
- net CH5: now also U12.2 (V_{OUT})
- net CH6: now reaches U11.7 (CH6)
- net CH6: now also RV2.2
- net CH7: now reaches U11.8 (CH7)
- net CH7: now also R99.1, RP1.2
- no-connect marks 0 -> 1
