File: 8051 Development Board v2/INT.kicad_sch (KiCad schematic)
At the start: 4 parts, among them SW2 SW_Push_Dual, SW3 SW_Push_Dual

Commit message: nets
Parts:
- C6, C7: footprint Capacitor_SMD:C_1206_3216Metric_Pad1.33x1.80mm_HandSolder -> Capacitor_SMD:C_1206_3216Metric
Changed lines of the file:
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@@
 	(wire
 		(pts
-			(xy 134.62 71.12) (xy 134.62 90.17)
+			(xy 134.62 76.2) (xy 134.62 90.17)
 		)
 		(stroke
@@
 	(wire
 		(pts
-			(xy 109.22 71.12) (xy 109.22 90.17)
+			(xy 109.22 76.2) (xy 109.22 90.17)
 		)
 		(stroke
@@
 	(hierarchical_label "P3.3"
 		(shape input)
-		(at 134.62 72.39 90)
+		(at 134.62 76.2 90)
 		(effects
 			(font
@@
 	(hierarchical_label "P3.2"
 		(shape input)
-		(at 109.22 72.39 90)
+		(at 109.22 76.2 90)
 		(effects
 			(font
@@
 			)
 		)
-		(property "Footprint" "Capacitor_SMD:C_1206_3216Metric_Pad1.33x1.80mm_HandSolder"
+		(property "Footprint" "Capacitor_SMD:C_1206_3216Metric"
 			(at 129.54 108.9152 0)
 			(effects
@@
 			)
 		)
-		(property "Footprint" "Capacitor_SMD:C_1206_3216Metric_Pad1.33x1.80mm_HandSolder"
+		(property "Footprint" "Capacitor_SMD:C_1206_3216Metric"
 			(at 96.52 108.9152 0)
 			(effects
@@
 		)
 		(instances
-			(project ""
+			(project "8051"
 				(path "/1fd5cb60-9043-4003-959b-0153e5ed66c7/3a1aa146-c8fa-4481-b1c3-c9a11d3b1e91"
 					(reference "C6")
@@
 		(dnp no)
 		(fields_autoplaced yes)
-		(property "Reference" "#PWR011"
+		(property "Reference" "#PWR0101"
 			(at 91.44 115.57 0)
 			(effects
@@
 		)
 		(instances
-			(project ""
+			(project "8051"
 				(path "/1fd5cb60-9043-4003-959b-0153e5ed66c7/3a1aa146-c8fa-4481-b1c3-c9a11d3b1e91"
-					(reference "#PWR011")
+					(reference "#PWR0101")
 					(unit 1)
 				)
