File: 8051 Development Board v2/buzzer.kicad_sch (KiCad schematic)
At the start: 4 parts, among them J21 Conn_01x01, Q8 BC548

Commit message: nets
Parts:
- R8: footprint ~ -> Resistor_SMD:R_1206_3216Metric
Changed lines of the file:
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@@
 			)
 		)
-		(property "Footprint" "~"
+		(property "Footprint" "Resistor_SMD:R_1206_3216Metric"
 			(at 134.62 94.488 90)
 			(effects
