File: 8051 Development Board v2/ledarray.kicad_sch (KiCad schematic)
At the start: 10 parts, among them J24 Conn_01x08

Commit message: nets
Parts:
- R16: footprint (none) -> Resistor_SMD:R_1206_3216Metric
Changed lines of the file:
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@@
 			)
 		)
-		(property "Footprint" ""
+		(property "Footprint" "Resistor_SMD:R_1206_3216Metric"
 			(at 124.46 132.08 0)
 			(effects
