File: 8051 Development Board v2/relays.kicad_sch (KiCad schematic)
At the start: 14 parts, among them J18 Conn_01x03, J19 Conn_01x03, J20 Conn_01x02, K1 RELAYPTH, K2 RELAYPTH, Q2 BC548, Q3 BC548

Commit message: nets
Parts:
- R5: footprint (none) -> Resistor_SMD:R_1206_3216Metric
- R6, R7: footprint ~ -> Resistor_SMD:R_1206_3216Metric
Other:
- moved on the sheet: D6, J19, K2, Q3, R6, R7
