File: 8051 Development Board v2/rtc.kicad_sch (KiCad schematic)
At the start: 6 parts, among them J23 Conn_01x03, U14 DS1307, U15 BATTERY, X1 CRYSTAL

Commit message: nets
Parts:
- R14, R15: footprint (none) -> Resistor_SMD:R_1206_3216Metric
Connections:
- net EBAT: now reaches U14.3 (VBAT), U15.1 (+)
Changed lines of the file:
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@@
+		)
+	)
+	(label "EBAT"
+		(at 175.26 100.33 0)
+		(effects
+			(font
+				(size 1.524 1.524)
+			)
+			(justify left bottom)
 		)
 	)
@@
 			)
 		)
-		(property "Footprint" ""
+		(property "Footprint" "Resistor_SMD:R_1206_3216Metric"
 			(at 129.54 87.63 0)
 			(effects
@@
 			)
 		)
-		(property "Footprint" ""
+		(property "Footprint" "Resistor_SMD:R_1206_3216Metric"
 			(at 124.46 87.63 0)
 			(effects
