File: 8051 Development Board v2/8051.kicad_sch (KiCad schematic)
At the start: 10 parts, among them J1 Conn_01x08, J3 Conn_01x08, J4 Conn_01x08, J5 Conn_01x08, U1 AT89S51-24PU, Y1 ABL-11.0592MHZ-B1U-T

Commit message: ultra
Parts:
- added RN10, RN11: R_Network08_US, Resistor_THT:R_Array_SIP9, symbol Device:R_Network08_US
- C2: value 30pF -> 22pF
- C3: value 30pF -> 2pF
Connections:
- net +5V: now also RN10.1 (common), RN11.1 (common)
- net P2.0: now also J4.8 (Pin_8), RN10.2 (R1); no longer J4.1 (Pin_1)
- net P2.1: now also J4.7 (Pin_7), RN10.3 (R2); no longer J4.2 (Pin_2)
- net P2.2: now also J4.6 (Pin_6), RN10.4 (R3); no longer J4.3 (Pin_3)
- net P2.3: now also J4.5 (Pin_5), RN10.5 (R4); no longer J4.4 (Pin_4)
- net P2.4: now also J4.4 (Pin_4), RN10.6 (R5); no longer J4.5 (Pin_5)
- net P2.5: now also J4.3 (Pin_3), RN10.7 (R6); no longer J4.6 (Pin_6)
- net P2.6: now also J4.2 (Pin_2), RN10.8 (R7); no longer J4.7 (Pin_7)
- net P2.7: now also J4.1 (Pin_1), RN10.9 (R8); no longer J4.8 (Pin_8)
- net P3.0: now also RN11.9 (R8)
- net P3.1: now also RN11.8 (R7)
- net P3.2: now also RN11.7 (R6)
- net P3.3: now also RN11.6 (R5)
- net P3.4: now also RN11.5 (R4)
- net P3.5: now also RN11.4 (R3)
- net P3.6: now also RN11.3 (R2)
- net P3.7: now also RN11.2 (R1)
- net P1.5 renamed MOSI
- net P1.6 renamed MISO
Other:
- added sheet 8-LED_ARRAY (ledarray.kicad_sch)
- added sheet ADC (ADC.kicad_sch)
- added sheet ADC_POT (adcpot.kicad_sch)
- added sheet BUZZER (buzzer.kicad_sch)
- added sheet DIP_SWITCHES (dipswitches.kicad_sch)
- added sheet EEPROM (eeprom.kicad_sch)
- added sheet LIGHT_SENSOR (lightsensor.kicad_sch)
- added sheet MOTOR_DRIVER (motordriver.kicad_sch)
- added sheet RELAYS (relays.kicad_sch)
- added sheet RTC (rtc.kicad_sch)
- added sheet TEMP_SENSOR (tempsensor.kicad_sch)
- moved on the sheet: C1, C2, C3, J1, J3, J4, J5, RN1, U1, Y1

Commit message: nets
Parts:
- C1, C2, C3: footprint Capacitor_SMD:C_1206_3216Metric_Pad1.33x1.80mm_HandSolder -> Capacitor_SMD:C_1206_3216Metric
Other:
- removed sheet ADC_POT
- removed sheet LIGHT_SENSOR
- removed sheet TEMP_SENSOR
- added sheet USB (USB.kicad_sch)
Changed lines of the file:
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@@
+	(wire
+		(pts
+			(xy 46.99 81.28) (xy 54.61 81.28)
+		)
+		(stroke
+			(width 0)
+			(type default)
+		)
+	)
 	(wire
 		(pts
@@
 	(wire
 		(pts
+			(xy 46.99 86.36) (xy 54.61 86.36)
+		)
+		(stroke
+			(width 0)
+			(type default)
+		)
+	)
+	(wire
+		(pts
 			(xy 168.91 118.11) (xy 175.26 118.11)
 		)
@@
 		)
 	)
+	(label "P3.1"
+		(at 54.61 86.36 180)
+		(effects
+			(font
+				(size 1.27 1.27)
+			)
+			(justify right bottom)
+		)
+	)
 	(label "P0.5"
 		(at 168.91 110.49 0)
@@
 			)
 			(justify left bottom)
+		)
+	)
+	(label "P3.0"
+		(at 54.61 81.28 180)
+		(effects
+			(font
+				(size 1.27 1.27)
+			)
+			(justify right bottom)
 		)
 	)
@@
 			)
 		)
-		(property "Footprint" "Capacitor_SMD:C_1206_3216Metric_Pad1.33x1.80mm_HandSolder"
+		(property "Footprint" "Capacitor_SMD:C_1206_3216Metric"
 			(at 94.9452 166.37 0)
 			(effects
@@
 			)
 		)
-		(property "Footprint" "Capacitor_SMD:C_1206_3216Metric_Pad1.33x1.80mm_HandSolder"
+		(property "Footprint" "Capacitor_SMD:C_1206_3216Metric"
 			(at 65.0748 166.37 0)
 			(effects
@@
 			)
 		)
-		(property "Footprint" "Capacitor_SMD:C_1206_3216Metric_Pad1.33x1.80mm_HandSolder"
+		(property "Footprint" "Capacitor_SMD:C_1206_3216Metric"
 			(at 162.2552 80.01 0)
 			(effects
@@
 	)
 	(sheet
-		(at 171.45 20.32)
-		(size 17.78 12.7)
-		(exclude_from_sim no)
-		(in_bom yes)
-		(on_board yes)
-		(dnp no)
-		(fields_autoplaced yes)
-		(stroke
-			(width 0.1524)
-			(type solid)
-		)
-		(fill
-			(color 0 0 0 0.0000)
-		)
-		(property "Sheetname" "TEMP_SENSOR"
-			(at 171.45 19.6084 0)
-			(effects
-				(font
-					(size 1.27 1.27)
-				)
-				(justify left bottom)
-			)
-		)
-		(property "Sheetfile" "tempsensor.kicad_sch"
-			(at 171.45 33.6046 0)
-			(effects
-				(font
-					(size 1.27 1.27)
-				)
-				(justify left top)
-			)
-		)
-		(instances
-			(project "8051"
-				(path "/1fd5cb60-9043-4003-959b-0153e5ed66c7"
-					(page "9")
-				)
-			)
-		)
-	)
-	(sheet
 		(at 113.03 20.32)
 		(size 17.78 12.7)
@@
 	)
 	(sheet
-		(at 200.66 20.32)
-		(size 17.78 12.7)
-		(exclude_from_sim no)
-		(in_bom yes)
-		(on_board yes)
-		(dnp no)
-		(fields_autoplaced yes)
-		(stroke
-			(width 0.1524)
-			(type solid)
-		)
-		(fill
-			(color 0 0 0 0.0000)
-		)
-		(property "Sheetname" "ADC_POT"
-			(at 200.66 19.6084 0)
-			(effects
-				(font
-					(size 1.27 1.27)
-				)
-				(justify left bottom)
-			)
-		)
-		(property "Sheetfile" "adcpot.kicad_sch"
-			(at 200.66 33.6046 0)
-			(effects
-				(font
-					(size 1.27 1.27)
-				)
-				(justify left top)
-			)
-		)
-		(instances
-			(project "8051"
-				(path "/1fd5cb60-9043-4003-959b-0153e5ed66c7"
-					(page "10")
-				)
-			)
-		)
-	)
-	(sheet
-		(at 229.87 20.32)
-		(size 17.78 12.7)
-		(exclude_from_sim no)
-		(in_bom yes)
-		(on_board yes)
-		(dnp no)
-		(fields_autoplaced yes)
-		(stroke
-			(width 0.1524)
-			(type solid)
-		)
-		(fill
-			(color 0 0 0 0.0000)
-		)
-		(property "Sheetname" "LIGHT_SENSOR"
-			(at 229.87 19.6084 0)
-			(effects
-				(font
-					(size 1.27 1.27)
-				)
-				(justify left bottom)
-			)
-		)
-		(property "Sheetfile" "lightsensor.kicad_sch"
-			(at 229.87 33.6046 0)
-			(effects
-				(font
-					(size 1.27 1.27)
-				)
-				(justify left top)
-			)
-		)
-		(instances
-			(project "8051"
-				(path "/1fd5cb60-9043-4003-959b-0153e5ed66c7"
-					(page "11")
-				)
-			)
-		)
-	)
-	(sheet
 		(at 52.07 20.32)
 		(size 17.78 12.7)
@@
 	)
 	(sheet
-		(at 200.66 48.26)
+		(at 171.45 20.32)
 		(size 17.78 12.7)
 		(exclude_from_sim no)
@@
 		)
 		(property "Sheetname" "MOTOR_DRIVER"
-			(at 200.66 47.5484 0)
+			(at 171.45 19.6084 0)
 			(effects
 				(font
@@
 		)
 		(property "Sheetfile" "motordriver.kicad_sch"
-			(at 200.66 61.5446 0)
+			(at 171.45 33.6046 0)
 			(effects
 				(font
@@
 				)
 			)
+		)
+	)
+	(sheet
+		(at 29.21 77.47)
+		(size 17.78 12.7)
+		(exclude_from_sim no)
+		(in_bom yes)
+		(on_board yes)
+		(dnp no)
+		(fields_autoplaced yes)
+		(stroke
+			(width 0.1524)
+			(type solid)
+		)
+		(fill
+			(color 0 0 0 0.0000)
+		)
+		(property "Sheetname" "USB"
+			(at 29.21 76.7584 0)
+			(effects
+				(font
+					(size 1.27 1.27)
+				)
+				(justify left bottom)
+			)
+		)
+		(property "Sheetfile" "USB.kicad_sch"
+			(at 29.21 90.7546 0)
+			(effects
+				(font
+					(size 1.27 1.27)
+				)
+				(justify left top)
+			)
+		)
+		(pin "TXD" input
+			(at 46.99 86.36 0)
+			(effects
+				(font
+					(size 1.27 1.27)
+				)
+				(justify right)
+			)
+		)
+		(pin "RXD" input
+			(at 46.99 81.28 0)
+			(effects
+				(font
+					(size 1.27 1.27)
+				)
+				(justify right)
+			)
+		)
+		(instances
+			(project "8051"
+				(path "/1fd5cb60-9043-4003-959b-0153e5ed66c7"
+					(page "10")
+				)
+			)

Commit message: usb
Other:
- note added: "REMOVE PULL UPS??"
Changed lines of the file:
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@@
 		(company "Momchil Kolev")
+	)
+	(text "REMOVE PULL UPS??"
+		(exclude_from_sim no)
+		(at 118.364 187.452 0)
+		(effects
+			(font
+				(size 5.08 5.08)
+			)
+		)
 	)
 	(junction
